Commit message: Fixed Aruco detection issues

File: rsc/car/car.urdf (robot description, URDF)
Before this commit: robot husky_robot, 13 links, 12 joints
Links:
- link aruco: geometry visual mesh filename=meshes/Aruco.stl scale=0.016 0.002 0.016
- link aruco_base: geometry visual box size=1.1 1.1 0.01
Joints:
- joint b_to_aruco: origin xyz=0 0 0.001 rpy=0 0 0 -> xyz=0 0 -0.05 rpy=0 0 0
